File: hw/xplorer.sch (EAGLE design)
At the start: 112 parts, among them T2 BC817, T5 ZDT6790, U1 PCM5102APW, U2 BMP085, U3 AD8345, U4 MIC5233, U5 MAX2614, U6 RA08H1317M, U7 TPS7A4901, U8 MAX4478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

Commit message: correct pcb file structure
Parts:
- removed R35: 8k8, rcl:R-EU_R0603
- removed T5: ZDT6790, ZDT6790:ZDT6790
- removed X2, X6, X8: (no value), wirepad:SMD2
- added C36, C37: 8p, rcl:C-EUC0805K
- added Q1: IRLML6402, transistor-power:IRLML5203
- added R12, R7: (no value), rcl:R-EU_R0603
- added R17: 475R, rcl:R-EU_R0603
- added R18: 1k, rcl:R-EU_R0603
- added R8: (no value), rcl:R-EU_R2010
- added T1: (no value), transistor:BC817-16-NPN-SOT23-BEC
- added X25: (no value), pinhead:PINHD-2X5
- added X7: (no value), wirepad:SMD2
- C11, C40: device rcl:C-EUC0603 -> rcl:C-EUC0805
- C20, C21: device rcl:C-EUC1812 -> rcl:C-EUC0805K
- H1, H2: value (none) -> PL006-WCR12; device led:LEDCHIPLED_0603 -> led:PL006-WCR12
- R11, R16: device rcl:R-EU_R0402 -> rcl:R-EU_R0603
- U2: value BMP085 -> SI570; device SparkFun:BMP085 -> silabs:SI570
Connections:
- removed net $234567898765: T5G$2.C1, T5G$2.C2, X2.P
- removed net N$31: R11.1, X1.GPIO18
- removed net N$55: R35.1, T5G$2.B
- new net HEAD: R17.1, X25.5
- new net N$13: R7.2, U2.SDA
- new net N$25: R12.1, R13.1, U7.EN
- new net N$27: R17.2, R18.2, X1.GPIO4,GPCLK0
- new net REL: Q1.D, X25.3
- new net STAT: H2.A, X1.GPIO10_MOSI
- new net VLA: C19.1, C20.1, C37.1, L1.1
- net +12V: now also Q1.S, X25.1; no longer T5G$2.E
- net +3V3: now also R8.1, X7.P; no longer C35.1, U2.VDDA, U2.VDDD
- net +5V: now also X25.7; no longer X8.P
- net GND: now also C36.2, C37.2, R11.1, R18.1, T1.E, X25.2, X25.4, X25.6, X25.8; no longer H2.C, T5G$1.E
- net LO: now also U2.CLK+; no longer X1.GPIO4,GPCLK0
- net N$14: now also C36.1
- net N$16: now also H2.C; no longer H2.A
- net N$19: now also C35.1, R8.2, U2.OE, U2.VDD; no longer C19.1, C20.1, L1.1
- net N$42: now also T1.B; no longer T5G$1.B
- net N$54: now also Q1.G, T1.C; no longer R35.2, T5G$1.C1, T5G$1.C2
- net N$66: now also X1.GPIO11_SCLK; no longer X1.GPIO27
- net PA_EN: now also R12.2, X1.GPIO7,SPI0_CE1; no longer R13.1, U7.EN, X1.GPIO22
- net PRE_EN: now also X1.GPIO8,SPI0_CE0; no longer X1.GPIO11_SCLK
- net REL_FB: now also X25.9; no longer X6.P
- net SDA: now also R7.1; no longer U2.SDA
Other:
- note added: "Temp"
- note removed: "T5"
- note removed: "ZDT6790"
